File: Quackboard_V0.kicad_sch (KiCad schematic)
At the start: 153 parts, among them J1 USB_C_Receptacle_USB2.0_16P, SW1 SW_Push, SW2 SW_SPDT, U1 STM32G0B1CBTx, U2 SRV05-4, U3 XC6206P332MR

Commit message: updated all files
Parts:
- removed D1, D10, D11, D12, D13, D14, D15, D16, D17, D18, D19, D2, D20, D21, D22, D23, D24, D25, D26, D27, D28, D29, D3, D30, D31, D32, D33, D34, D35, D36, D37, D38, D39, D4, D40, D41, D42, D44, D45, D46, D47, D49, D5, D50, D51, D52, D54, D56, D57, D58, D6, D60, D62, D64, D65, D66, D67, D68, D69, D7, D70, D71, D72, D73, D74, D75, D8, D9: 1N4148W, Diode_SMD:D_SOD-123, symbol Device:D
- removed MX1, MX10, MX11, MX12, MX13, MX14, MX15, MX16, MX17, MX18, MX19, MX2, MX20, MX21, MX22, MX23, MX24, MX25, MX26, MX27, MX28, MX29, MX3, MX30, MX31, MX32, MX33, MX34, MX35, MX36, MX37, MX38, MX39, MX4, MX40, MX41, MX42, MX44, MX45, MX46, MX47, MX49, MX5, MX50, MX51, MX52, MX54, MX56, MX57, MX58, MX6, MX60, MX62, MX64, MX65, MX66, MX67, MX68, MX69, MX7, MX70, MX71, MX72, MX73, MX74, MX75, MX8, MX9: MX_Keyswitch, symbol Switch:SW_Push
- removed U2: SRV05-4, PCM_marbastlib-various:SOT-23-6-routable, symbol PCM_marbastlib-various:SRV05-4
- added U4: SRV05-4, Package_TO_SOT_SMD:SOT-23-6, symbol Power_Protection:SRV05-4
- C1: renamed from C7; footprint Diode_SMD:D_SOD-123 -> Capacitor_SMD:C_0805_2012Metric
- SW1: renamed from SW2; footprint Button_Switch_SMD:SW_SPDT_PCM12 -> Button_Switch_THT:SW_Slide_SPDT_Straight_CK_OS102011MS2Q
- SW2: renamed from SW1; footprint (none) -> Button_Switch_SMD:SW_SPST_TL3342
- renumbered C6 to C2, C1 to C3, C2 to C4, C3 to C6, C4 to C7, R2 to R1, R1 to R2, U3 to U2, U1 to U3
Connections:
- net +5V: now also U4.5 (VP)
- net COL0: now also U3.26 (PB14)
- net COL1: now also U3.27 (PB15)
- net COL10: now also U3.23 (PB11)
- net COL11: now also U3.22 (PB10)
- net COL12: now also U3.21 (PB2)
- net COL13: now also U3.20 (PB1)
- net COL14: now also U3.19 (PB0)
- net COL2: now also U3.28 (PA8)
- net COL3: now also U3.29 (PA9/UCPD1_DBCC1)
- net COL4: now also U3.11 (PA0)
- net COL5: now also U3.12 (PA1)
- net COL6: now also U3.24 (PB12)
- net COL7: now also U3.15 (PA4)
- net COL8: now also U3.16 (PA5)
- net COL9: now also U3.17 (PA6)
- net D+: now also U4.1 (IO1)
- net D-: now also U4.3 (IO2)
- net GND: now also U4.2 (VN)
- net ROW0: now also U3.48 (PB9)
- net ROW1: now also U3.47 (PB8)
- net ROW2: now also U3.46 (PB7)
- net ROW3: now also U3.45 (PB6)
- net ROW4: now also U3.25 (PB13)
- net COL15: now reaches U3.18 (PA7)
- no-connect marks 2 -> 23
Other:
- added sheet Switch Matrix (matrix.kicad_sch)
